File: Schematics/Barometer.kicad_sch (KiCad schematic)
At the start: 4 parts, among them U6 MPL3115A2R1

Commit message: output files got quote
Parts:
- C20, C21, C22: LCSC (none) -> C49678; LCSC Part C49678 -> (none)
- U6: LCSC (none) -> C54429; LCSC Part C54429 -> (none)
Changed lines of the file:
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@@
-			)
-		)
-		(property "LCSC Part" "C49678"
-			(at 100.33 81.28 0)
-			(effects
-				(font
-					(size 1.27 1.27)
-				)
-				(hide yes)
 			)
 		)
@@
 		)
 		(property "Purchase-URL" ""
+			(at 100.33 81.28 0)
+			(effects
+				(font
+					(size 1.27 1.27)
+				)
+				(hide yes)
+			)
+		)
+		(property "LCSC" "C49678"
 			(at 100.33 81.28 0)
 			(effects
@@
 			)
 		)
-		(property "LCSC Part" "C54429"
-			(at 137.16 82.55 0)
-			(effects
-				(font
-					(size 1.27 1.27)
-				)
-				(hide yes)
-			)
-		)
 		(property "Description_1" ""
 			(at 137.16 82.55 0)
@@
 		)
 		(property "Purchase-URL" ""
+			(at 137.16 82.55 0)
+			(effects
+				(font
+					(size 1.27 1.27)
+				)
+				(hide yes)
+			)
+		)
+		(property "LCSC" "C54429"
 			(at 137.16 82.55 0)
 			(effects
@@
 			)
 		)
-		(property "LCSC Part" "C49678"
-			(at 110.49 81.28 0)
-			(effects
-				(font
-					(size 1.27 1.27)
-				)
-				(hide yes)
-			)
-		)
 		(property "Description_1" ""
 			(at 110.49 81.28 0)
@@
 		)
 		(property "Purchase-URL" ""
+			(at 110.49 81.28 0)
+			(effects
+				(font
+					(size 1.27 1.27)
+				)
+				(hide yes)
+			)
+		)
+		(property "LCSC" "C49678"
 			(at 110.49 81.28 0)
 			(effects
@@
 			)
 		)
-		(property "LCSC Part" "C49678"
-			(at 119.38 82.55 0)
-			(effects
-				(font
-					(size 1.27 1.27)
-				)
-				(hide yes)
-			)
-		)
 		(property "Description_1" ""
 			(at 119.38 82.55 0)
@@
 			(at 119.38 82.55 0)
 			(effects
+				(font
+					(size 1.27 1.27)
+				)
+				(hide yes)
+			)
+		)
+		(property "LCSC" "C49678"
+			(at 119.38 82.55 0)
+			(effects
