File: Schematics/Can_transceiver.kicad_sch (KiCad schematic)
At the start: 6 parts, among them U2 SN65HVD230

Commit message: output files got quote
Parts:
- C17: LCSC (none) -> C49678; LCSC Part C49678 -> (none)
- CAN_IN1, CAN_OUT1: LCSC (none) -> C17644051; LCSC Part C17644051 -> (none)
- JP1: now not fitted
- R8: LCSC (none) -> C269726; LCSC Part C269726 -> (none)
- U2: LCSC (none) -> C1543812; LCSC Part C1543812 -> (none)
Changed lines of the file:
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@@
 		(in_bom no)
 		(on_board yes)
-		(dnp no)
+		(dnp yes)
 		(property "Reference" "JP1"
 			(at 161.29 101.346 0)
@@
 			)
 		)
-		(property "LCSC Part" "C17644051"
-			(at 198.12 85.09 0)
-			(effects
-				(font
-					(size 1.27 1.27)
-				)
-				(hide yes)
-			)
-		)
 		(property "Description_1" ""
 			(at 198.12 85.09 0)
@@
 		)
 		(property "Purchase-URL" ""
+			(at 198.12 85.09 0)
+			(effects
+				(font
+					(size 1.27 1.27)
+				)
+				(hide yes)
+			)
+		)
+		(property "LCSC" "C17644051"
 			(at 198.12 85.09 0)
 			(effects
@@
 			)
 		)
-		(property "LCSC Part" "C49678"
-			(at 101.6 90.17 0)
-			(effects
-				(font
-					(size 1.27 1.27)
-				)
-				(hide yes)
-			)
-		)
 		(property "Description_1" ""
 			(at 101.6 90.17 0)
@@
 		)
 		(property "Purchase-URL" ""
+			(at 101.6 90.17 0)
+			(effects
+				(font
+					(size 1.27 1.27)
+				)
+				(hide yes)
+			)
+		)
+		(property "LCSC" "C49678"
 			(at 101.6 90.17 0)
 			(effects
@@
 			)
 		)
-		(property "LCSC Part" "C269726"
-			(at 156.21 90.17 0)
-			(effects
-				(font
-					(size 1.27 1.27)
-				)
-				(hide yes)
-			)
-		)
 		(property "Description_1" ""
 			(at 156.21 90.17 0)
@@
 		)
 		(property "Purchase-URL" ""
+			(at 156.21 90.17 0)
+			(effects
+				(font
+					(size 1.27 1.27)
+				)
+				(hide yes)
+			)
+		)
+		(property "LCSC" "C269726"
 			(at 156.21 90.17 0)
 			(effects
@@
 			)
 		)
-		(property "LCSC Part" "C1543812"
-			(at 140.97 88.9 0)
-			(effects
-				(font
-					(size 1.27 1.27)
-				)
-				(hide yes)
-			)
-		)
 		(property "Description_1" ""
 			(at 140.97 88.9 0)
@@
 		)
 		(property "Purchase-URL" ""
+			(at 140.97 88.9 0)
+			(effects
+				(font
+					(size 1.27 1.27)
+				)
+				(hide yes)
+			)
+		)
+		(property "LCSC" "C1543812"
 			(at 140.97 88.9 0)
 			(effects
@@
 			)
 		)
-		(property "LCSC Part" "C17644051"
-			(at 198.12 93.98 0)
-			(effects
-				(font
-					(size 1.27 1.27)
-				)
-				(hide yes)
-			)
-		)
 		(property "Description_1" ""
 			(at 198.12 93.98 0)
@@
 			(at 198.12 93.98 0)
 			(effects
+				(font
+					(size 1.27 1.27)
+				)
+				(hide yes)
+			)
+		)
+		(property "LCSC" "C17644051"
+			(at 198.12 93.98 0)
+			(effects
