File: Schematics/Drogue.kicad_sch (KiCad schematic)
At the start: 6 parts, among them J4 Pyro, Q2 BSC098N10NS5

Commit message: output files got quote
Parts:
- J4: LCSC (none) -> C17644051; LCSC Part C17644051 -> (none)
- Q2: value BSC098N10NS5 -> IRLML2502TRPBF; footprint Package_TO_SOT_SMD:SOT-23-5 -> myFootprints:SOT23; symbol Transistor_FET:BSC098N10NS5 -> Transistor_FET:Q_NMOS_DGS; LCSC (none) -> C2589; LCSC Part C534398 -> (none)
- R10: LCSC (none) -> C84376; LCSC Part C84376 -> (none)
- R11: LCSC (none) -> C17819; LCSC Part C96346 -> (none)
- R12: LCSC (none) -> C2933415; LCSC Part C2933415 -> (none)
- R9: LCSC (none) -> C17408; LCSC Part C17408 -> (none)
Connections:
- net GND: no longer Q2.1 (S), Q2.3 (S)
- net at J4.2 (Pin_2), R11.2: now also Q2.3 (S); no longer Q2.5 (D)
- net at R10.1, R9.1: now also Q2.1 (D); no longer Q2.4 (G)
Other:
- moved on the sheet: Q2, R10, R9
