File: Schematics/FlashMemory.kicad_sch (KiCad schematic)
At the start: 4 parts, among them U8 W25Q128JVP

Commit message: output files got quote
Parts:
- C26: LCSC (none) -> C49678; LCSC Part C49678 -> (none)
- R17, R18: LCSC (none) -> C84376; LCSC Part C84376 -> (none)
- U8: LCSC (none) -> C190862; LCSC Part C190862 -> (none)
Changed lines of the file:
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@@
 			)
 		)
-		(property "LCSC Part" "C190862"
+		(property "LCSC" "C190862"
 			(at 127 85.09 0)
 			(effects
@@
 			)
 		)
-		(property "LCSC Part" "C49678"
+		(property "LCSC" "C49678"
 			(at 134.62 63.5 90)
 			(effects
@@
 			)
 		)
-		(property "LCSC Part" "C84376"
+		(property "LCSC" "C84376"
 			(at 109.22 93.98 0)
 			(effects
@@
 			)
 		)
-		(property "LCSC Part" "C84376"
+		(property "LCSC" "C84376"
 			(at 100.33 91.44 0)
 			(effects
