File: Schematics/GPS1.kicad_sch (KiCad schematic)
At the start: 2 parts, among them J5 Conn_01x05_Pin, J6 Conn_01x05_Pin

Commit message: output files got quote
Parts:
- J5, J6: LCSC (none) -> C157991; LCSC Part C157991 -> (none)
Changed lines of the file:
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@@
-			)
-		)
-		(property "LCSC Part" "C157991"
-			(at 132.08 95.25 0)
-			(effects
-				(font
-					(size 1.27 1.27)
-				)
-				(hide yes)
 			)
 		)
@@
 		)
 		(property "Purchase-URL" ""
+			(at 132.08 95.25 0)
+			(effects
+				(font
+					(size 1.27 1.27)
+				)
+				(hide yes)
+			)
+		)
+		(property "LCSC" "C157991"
 			(at 132.08 95.25 0)
 			(effects
@@
 			)
 		)
-		(property "LCSC Part" "C157991"
-			(at 132.08 118.11 0)
-			(effects
-				(font
-					(size 1.27 1.27)
-				)
-				(hide yes)
-			)
-		)
 		(property "Description_1" ""
 			(at 132.08 118.11 0)
@@
 			(at 132.08 118.11 0)
 			(effects
+				(font
+					(size 1.27 1.27)
+				)
+				(hide yes)
+			)
+		)
+		(property "LCSC" "C157991"
+			(at 132.08 118.11 0)
+			(effects
