File: Schematics/IMU.kicad_sch (KiCad schematic)
At the start: 4 parts, among them U7 LSM6DS3TR-C

Commit message: output files got quote
Parts:
- C23, C24, C25: LCSC (none) -> C49678; LCSC Part C49678 -> (none)
- U7: LCSC (none) -> C967633; LCSC Part C967633 -> (none)
Changed lines of the file:
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@@
-			)
-		)
-		(property "LCSC Part" "C967633"
-			(at 139.7 113.03 0)
-			(effects
-				(font
-					(size 1.27 1.27)
-				)
-				(hide yes)
 			)
 		)
@@
 		)
 		(property "Purchase-URL" ""
+			(at 139.7 113.03 0)
+			(effects
+				(font
+					(size 1.27 1.27)
+				)
+				(hide yes)
+			)
+		)
+		(property "LCSC" "C967633"
 			(at 139.7 113.03 0)
 			(effects
@@
 			)
 		)
-		(property "LCSC Part" "C49678"
-			(at 129.54 66.04 0)
-			(effects
-				(font
-					(size 1.27 1.27)
-				)
-				(hide yes)
-			)
-		)
 		(property "Description_1" ""
 			(at 129.54 66.04 0)
@@
 		)
 		(property "Purchase-URL" ""
+			(at 129.54 66.04 0)
+			(effects
+				(font
+					(size 1.27 1.27)
+				)
+				(hide yes)
+			)
+		)
+		(property "LCSC" "C49678"
 			(at 129.54 66.04 0)
 			(effects
@@
 			)
 		)
-		(property "LCSC Part" "C49678"
-			(at 129.54 78.74 0)
-			(effects
-				(font
-					(size 1.27 1.27)
-				)
-				(hide yes)
-			)
-		)
 		(property "Description_1" ""
 			(at 129.54 78.74 0)
@@
 		)
 		(property "Purchase-URL" ""
+			(at 129.54 78.74 0)
+			(effects
+				(font
+					(size 1.27 1.27)
+				)
+				(hide yes)
+			)
+		)
+		(property "LCSC" "C49678"
 			(at 129.54 78.74 0)
 			(effects
@@
 			)
 		)
-		(property "LCSC Part" "C49678"
-			(at 153.67 78.74 0)
-			(effects
-				(font
-					(size 1.27 1.27)
-				)
-				(hide yes)
-			)
-		)
 		(property "Description_1" ""
 			(at 153.67 78.74 0)
@@
 			(at 153.67 78.74 0)
 			(effects
+				(font
+					(size 1.27 1.27)
+				)
+				(hide yes)
+			)
+		)
+		(property "LCSC" "C49678"
+			(at 153.67 78.74 0)
+			(effects
