File: Schematics/LoRa.kicad_sch (KiCad schematic)
At the start: 2 parts, among them J7 Conn_Coaxial_Small, U5 RFM95W-915S2

Commit message: output files got quote
Parts:
- J7: LCSC (none) -> C3172376; LCSC Part C3172376 -> (none)
- U5: LCSC (none) -> C2844473; LCSC Part C2844473 -> (none)
Changed lines of the file:
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@@
-			)
-		)
-		(property "LCSC Part" "C3172376"
-			(at 176.53 76.2 0)
-			(effects
-				(font
-					(size 1.27 1.27)
-				)
-				(hide yes)
 			)
 		)
@@
 		)
 		(property "Purchase-URL" ""
+			(at 176.53 76.2 0)
+			(effects
+				(font
+					(size 1.27 1.27)
+				)
+				(hide yes)
+			)
+		)
+		(property "LCSC" "C3172376"
 			(at 176.53 76.2 0)
 			(effects
@@
 			)
 		)
-		(property "LCSC Part" "C2844473"
-			(at 130.81 83.82 0)
-			(effects
+		(property "LCSC" "C2844473"
+			(at 130.81 83.82 0)
+			(effects
