File: Schematics/power.kicad_sch (KiCad schematic)
At the start: 6 parts, among them U3 PowerIn, U4 LDL1117-3.3

Commit message: output files got quote
Parts:
- C18: LCSC (none) -> C49678; LCSC Part C49678 -> (none)
- C19: LCSC (none) -> C2932476; LCSC Part C98192 -> (none)
- D2, D3: LCSC (none) -> C113936; LCSC Part C113936 -> (none)
- U3: LCSC (none) -> C17644051; LCSC Part C17644051 -> (none)
- U4: LCSC (none) -> C435835; LCSC Part C435835 -> (none)
Changed lines of the file:
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@@
-			)
-		)
-		(property "LCSC Part" "C17644051"
-			(at 130.81 53.34 0)
-			(effects
-				(font
-					(size 1.27 1.27)
-				)
-				(hide yes)
 			)
 		)
@@
 		)
 		(property "Purchase-URL" ""
+			(at 130.81 53.34 0)
+			(effects
+				(font
+					(size 1.27 1.27)
+				)
+				(hide yes)
+			)
+		)
+		(property "LCSC" "C17644051"
 			(at 130.81 53.34 0)
 			(effects
@@
 			)
 		)
-		(property "LCSC" ""
+		(property "LCSC" "C113936"
 			(at 78.74 76.2 90)
 			(effects
@@
 		)
 		(property "Description_1" ""
-			(at 78.74 76.2 90)
-			(effects
-				(font
-					(size 1.27 1.27)
-				)
-				(hide yes)
-			)
-		)
-		(property "LCSC Part" "C113936"
 			(at 78.74 76.2 90)
 			(effects
@@
 			)
 		)
-		(property "LCSC" ""
+		(property "LCSC" "C113936"
 			(at 96.52 76.2 90)
 			(effects
@@
 		)
 		(property "Description_1" ""
-			(at 96.52 76.2 90)
-			(effects
-				(font
-					(size 1.27 1.27)
-				)
-				(hide yes)
-			)
-		)
-		(property "LCSC Part" "C113936"
 			(at 96.52 76.2 90)
 			(effects
@@
 			)
 		)
-		(property "LCSC" ""
+		(property "LCSC" "C435835"
 			(at 159.766 94.742 0)
 			(effects
@@
 		)
 		(property "Description_1" ""
-			(at 151.13 100.33 0)
-			(effects
-				(font
-					(size 1.27 1.27)
-				)
-				(hide yes)
-			)
-		)
-		(property "LCSC Part" "C435835"
 			(at 151.13 100.33 0)
 			(effects
@@
 			)
 		)
-		(property "LCSC Part" "C98192"
-			(at 176.53 86.36 0)
-			(effects
-				(font
-					(size 1.27 1.27)
-				)
-				(hide yes)
-			)
-		)
 		(property "Description_1" ""
 			(at 176.53 86.36 0)
@@
 		)
 		(property "Purchase-URL" ""
+			(at 176.53 86.36 0)
+			(effects
+				(font
+					(size 1.27 1.27)
+				)
+				(hide yes)
+			)
+		)
+		(property "LCSC" "C2932476"
 			(at 176.53 86.36 0)
 			(effects
@@
 			)
 		)
-		(property "LCSC Part" "C49678"
-			(at 121.92 86.36 0)
-			(effects
-				(font
-					(size 1.27 1.27)
-				)
-				(hide yes)
-			)
-		)
 		(property "Description_1" ""
 			(at 121.92 86.36 0)
@@
 			(at 121.92 86.36 0)
 			(effects
+				(font
+					(size 1.27 1.27)
+				)
+				(hide yes)
+			)
+		)
+		(property "LCSC" "C49678"
+			(at 121.92 86.36 0)
+			(effects
