File: Schematics/pyro.kicad_sch (KiCad schematic)
At the start: 6 parts, among them J2 Pyro, Q1 BSC098N10NS5

Commit message: output files got quote
Parts:
- J2: LCSC (none) -> C17644051; LCSC Part C17644051 -> (none)
- Q1: value BSC098N10NS5 -> IRLML2502TRPBF; footprint Package_TO_SOT_SMD:SOT-23-5 -> myFootprints:SOT23; symbol Transistor_FET:BSC098N10NS5 -> Transistor_FET:Q_NMOS_DGS; LCSC (none) -> C2589; LCSC Part C534398 -> (none)
- R4: LCSC (none) -> C17408; LCSC Part C17408 -> (none)
- R5: LCSC (none) -> C84376; LCSC Part C84376 -> (none)
- R6: LCSC (none) -> C17819; LCSC Part C96346 -> (none)
- R7: LCSC (none) -> C2933415; LCSC Part C2933415 -> (none)
Connections:
- net GND: no longer Q1.1 (S), Q1.3 (S)
- net at J2.2 (Pin_2), R6.2: now also Q1.3 (S); no longer Q1.5 (D)
- net at R4.1, R5.1: now also Q1.1 (D); no longer Q1.4 (G)
Other:
- moved on the sheet: Q1, R4, R5
