File: Schematics/usb_type_c_sch.kicad_sch (KiCad schematic)
At the start: 4 parts, among them J2 USB_C_Receptacle_USB2.0_16P

Commit message: output files got quote
Parts:
- D4: LCSC (none) -> C13612; LCSC Part C13612 -> (none)
- J9: renamed from J2; LCSC (none) -> C165948; LCSC Part C165948 -> (none)
- R13, R14: LCSC (none) -> C27834; LCSC Part C27834 -> (none)
Changed lines of the file:
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@@
-			)
-		)
-		(property "LCSC Part" "C13612"
-			(at 162.56 73.66 0)
-			(effects
-				(font
-					(size 1.27 1.27)
-				)
-				(hide yes)
 			)
 		)
@@
 		)
 		(property "Purchase-URL" ""
+			(at 162.56 73.66 0)
+			(effects
+				(font
+					(size 1.27 1.27)
+				)
+				(hide yes)
+			)
+		)
+		(property "LCSC" "C13612"
 			(at 162.56 73.66 0)
 			(effects
@@
 			)
 		)
-		(property "LCSC Part" "C27834"
-			(at 186.69 66.04 0)
-			(effects
-				(font
-					(size 1.27 1.27)
-				)
-				(hide yes)
-			)
-		)
 		(property "Description_1" ""
 			(at 186.69 66.04 0)
@@
 		)
 		(property "Purchase-URL" ""
+			(at 186.69 66.04 0)
+			(effects
+				(font
+					(size 1.27 1.27)
+				)
+				(hide yes)
+			)
+		)
+		(property "LCSC" "C27834"
 			(at 186.69 66.04 0)
 			(effects
@@
 			)
 		)
-		(property "LCSC Part" "C27834"
-			(at 175.26 68.58 0)
-			(effects
-				(font
-					(size 1.27 1.27)
-				)
-				(hide yes)
-			)
-		)
 		(property "Description_1" ""
 			(at 175.26 68.58 0)
@@
 		)
 		(property "Purchase-URL" ""
+			(at 175.26 68.58 0)
+			(effects
+				(font
+					(size 1.27 1.27)
+				)
+				(hide yes)
+			)
+		)
+		(property "LCSC" "C27834"
 			(at 175.26 68.58 0)
 			(effects
@@
 		(dnp no)
 		(fields_autoplaced yes)
-		(property "Reference" "J2"
+		(property "Reference" "J9"
 			(at 107.95 49.53 0)
 			(effects
@@
 			)
 		)
-		(property "LCSC Part" "C165948"
+		(property "LCSC" "C165948"
 			(at 107.95 72.39 0)
 			(effects
@@
 			(project ""
 				(path "/6cb3dda3-5fe8-4715-b831-354360aa3199/105f27ec-5fab-44f4-a683-69b23a7486f0"
-					(reference "J2")
-					(unit 1)
-				)
+					(reference "J9")
+					(unit 1)
+				)
