File: Schematics/Accelerometer.kicad_sch (KiCad schematic)
At the start: 3 parts, among them U9 H3LIS100DL

Commit message: output files got quote
Parts:
- C27: LCSC (none) -> C49678; LCSC Part C49678 -> (none)
- C28: LCSC (none) -> C28323; LCSC Part C28323 -> (none)
- U9: LCSC (none) -> C2655068; LCSC Part C2655068 -> (none)
Changed lines of the file:
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@@
 			)
 		)
-		(property "LCSC Part" "C49678"
+		(property "LCSC" "C49678"
 			(at 156.21 82.55 0)
 			(effects
@@
 			)
 		)
-		(property "LCSC Part" "C2655068"
-			(at 105.41 100.584 0)
-			(effects
-				(font
-					(size 1.27 1.27)
-				)
-				(hide yes)
-			)
-		)
 		(property "Description_1" ""
 			(at 137.16 102.87 0)
@@
 		)
 		(property "Purchase-URL" ""
+			(at 137.16 102.87 0)
+			(effects
+				(font
+					(size 1.27 1.27)
+				)
+				(hide yes)
+			)
+		)
+		(property "LCSC" "C2655068"
 			(at 137.16 102.87 0)
 			(effects
@@
 			)
 		)
-		(property "LCSC Part" "C28323"
-			(at 168.91 82.55 0)
-			(effects
+		(property "LCSC" "C28323"
+			(at 168.91 82.55 0)
+			(effects

Commit message: finalized output files
Parts:
- U9: value H3LIS100DL -> H3LIS331DL; LCSC C2655068 -> C2655074
Changed lines of the file:
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@@
 			)
 		)
-		(property "Value" "H3LIS100DL"
+		(property "Value" "H3LIS331DL"
 			(at 132.588 88.392 0)
 			(effects
@@
 			)
 		)
-		(property "LCSC" "C2655068"
+		(property "LCSC" "C2655074"
 			(at 137.16 102.87 0)
 			(effects
