File: Schematics/MCU.kicad_sch (KiCad schematic)
At the start: 32 parts, among them J1 Microsemi_FlashPro-JTAG-10, Q3 BC817, U1 STM32F405RGT6, Y1 8mhz

Commit message: output files got quote
Parts:
- BZ1: LCSC (none) -> C96093; LCSC Part C96093 -> (none)
- C1, C10, C11, C12, C14, C2, C5, C6, C7: LCSC (none) -> C49678; LCSC Part C49678 -> (none)
- C13, C9: LCSC (none) -> C28323; LCSC Part C28323 -> (none)
- C15, C16: LCSC (none) -> C170109; LCSC Part C170109 -> (none)
- C3, C4: LCSC (none) -> C19110; LCSC Part C19110 -> (none)
- C8: LCSC (none) -> C98192; LCSC Part C98192 -> (none)
- D1: LCSC (none) -> C2827321; LCSC Part C2827321 -> (none)
- D6: LCSC (none) -> C191023; LCSC Part C191023 -> (none)
- FB1: LCSC (none) -> C85840; LCSC Part C85840 -> (none)
- J1: LCSC (none) -> C585350; LCSC Part C585350 -> (none)
- PowerLED1: LCSC (none) -> C965799; LCSC Part C965799 -> (none)
- Q3: LCSC (none) -> C39828; LCSC Part C39828 -> (none)
- R1, R20: LCSC (none) -> C84376; LCSC Part C84376 -> (none)
- R19: LCSC (none) -> C2907267; LCSC Part C2907267 -> (none)
- R2: LCSC (none) -> C96346; LCSC Part C96346 -> (none)
- R3: LCSC (none) -> C95781; LCSC Part C95781 -> (none)
- SW1: renamed from RSTSwitch1; LCSC (none) -> C49393646; LCSC Part C49393646 -> (none)
- SW2: renamed from BootSwitch1; LCSC (none) -> C49393646; LCSC Part C49393646 -> (none)
- U1: LCSC (none) -> C15742; LCSC Part C15742 -> (none)
- Y1: LCSC (none) -> C19723344; LCSC Part C19723344 -> (none)

Commit message: finalized output files
Parts:
- added R21, R22: 4.7k, Resistor_SMD:R_0805_2012Metric_Pad1.20x1.40mm_HandSolder, symbol Device:R
- C15, C16: LCSC C170109 -> C113825
- C8: LCSC C98192 -> C1779
Connections:
- net +3.3V: now also R21.2, R22.1
- net I2CSDA: now also R22.2
- net I2CSDL: now also R21.1
Other:
- note added: "Pullup resistors on I2C becuase devices control low (Open Drain)"
