File: Schematics/flightcomputer2.kicad_pcb (KiCad board)
At the start: 4 copper layers, 80 x 80 mm, 86 parts, among them J1 Microsemi_FlashPro-JTAG-10, J2 Pyro, J2 USB_C_Receptacle_USB2.0_16P, J4 Pyro, J5 Conn_01x05_Pin, J6 Conn_01x05_Pin, J7 Conn_Coaxial_Small, J8 Micro_SD_Card, Q1 BSC098N10NS5, Q2 BSC098N10NS5, Q3 BC817, U1 STM32F405RGT6, U2 SN65HVD230, U3 PowerIn, U4 LDL1117-3.3, U5 RFM95W-915S2, U6 MPL3115A2R1, U7 LSM6DS3TR-C, U8 W25Q128JVP, U9 H3LIS100DL, Y1 8mhz

Commit message: output files got quote
Parts:
- removed the J2 at (190.8, 99.5)
- added G***: LOGO, LOGO, F.Cu at (137.2, 88.9)
- added J9: USB_C_Receptacle_USB2.0_16P, Connector_USB:USB_C_Receptacle_HRO_TYPE-C-31-M-12, F.Cu at (190.8, 99.4)
- Q1, Q2: value BSC098N10NS5 -> IRLML2502TRPBF; footprint Package_TO_SOT_SMD:SOT-23-5 -> myFootprints:SOT23
- moved R9 3.71 mm to (137.9, 100.5)
- moved R6 3.46 mm to (121.4, 104.9)
- moved R7 3.46 mm to (121.4, 99.9)
- moved R10 2.75 mm to (138.0, 104.3), turned to -90 degrees
- moved Q2 2.02 mm to (135.2, 104.4)
- moved Q1 2.00 mm to (125.0, 104.8)
- moved R11 0.20 mm to (131.9, 104.7)
- renumbered RSTSwitch1 to SW1, BootSwitch1 to SW2
Connections:
- Q1 pad 1: GND -> Net-(Q1-D)
- Q1 pad 3: GND -> Net-(J2-Pin_2)
- Q2 pad 1: GND -> Net-(Q2-D)
- Q2 pad 3: GND -> Net-(J4-Pin_2)
- R10 pad 1: Net-(Q2-G) -> Net-(Q2-D)
- R4 pad 1: Net-(Q1-G) -> Net-(Q1-D)
- R5 pad 1: Net-(Q1-G) -> Net-(Q1-D)
- R9 pad 1: Net-(Q2-G) -> Net-(Q2-D)
Routing:
- net GND: track 171.7 -> 161.1 mm
- net /MCU/NRST: track 71.1 -> 78.3 mm
- net Net-(Q1-D): track 0.00 -> 4.79 mm
- net Net-(Q1-G): track 4.72 -> 0.00 mm
- net Net-(Q2-G): track 3.97 -> 0.00 mm
- net Net-(Q2-D): track 0.00 -> 3.69 mm
- net /Drogue/DrougeIgnite: track 60.0 -> 56.4 mm
- net /LoRa/sxNSS: track 44.6 -> 46.0 mm
- net +3.3V: track 119.2 -> 118.0 mm
- net /MCU/OSC IN: track 8.80 -> 7.84 mm
- net Net-(J2-Pin_2): track 8.75 -> 7.83 mm
- net /FlashSd/SDCLK: track 19.4 -> 20.2 mm
- net /LoRa/sxMIS0: track 42.7 -> 41.9 mm
- net /Drogue/DrougeADC: track 45.8 -> 46.5 mm
- net /MCU/D-: track 26.4 -> 25.8 mm
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Other:
- board text added: "Buttons"
- board text added: "CAN"
- board text added: "DROUGE"
- board text added: "GPS 1"
- board text added: "GPS 2"
- board text added: "JTAG"
- board text added: "NRST"
- board text added: "POWER IN"
- board text added: "PWR"
- board text added: "PYRO"
- board text added: "RST"
- board text added: "RX"
- board text added: "SWCLK"
- board text added: "SWDIO"
- board text added: "TX"
- board text added: "UTS Rocketry"
- board text added: "reetabass & ollie"
- board text removed: "Power"

Commit message: finalized output files
Parts:
- added R21: 4.7u, Resistor_SMD:R_0805_2012Metric_Pad1.20x1.40mm_HandSolder, F.Cu at (147.0, 66.7)
- added R22: 4.7u, Resistor_SMD:R_0805_2012Metric_Pad1.20x1.40mm_HandSolder, F.Cu at (148.9, 66.7)
Routing:
- net /Accelerometer/AccelerometerSDA: track 38.6 -> 46.1 mm
- net /Accelerometer/AccelerometerSCL: track 38.3 -> 43.5 mm
- net +3.3V: track 118.0 -> 120.7 mm, vias 26 -> 28
Other:
- board text removed: "NRST"
