File: Schematics/flightcomputer2.kicad_pcb (KiCad board)
At the start: 4 copper layers, 80 x 80 mm, 113 parts, among them J1 Microsemi_FlashPro-JTAG-10, J10 Pyro, J2 Pyro, J4 Drouge, J5 Conn_01x05_Pin, J6 Conn_01x05_Pin, J7 Conn_Coaxial_Small, J8 Micro_SD_Card, J9 USB_C_Receptacle_USB2.0_16P, Q1 IRLML2502TRPBF, Q2 IRLML2502TRPBF, Q3 BC817, Q4 IRLML2502TRPBF, Q6 Q_PMOS_GSD, SW1 SAMZO G4R0015010, SW2 SAMZO G4R0015010, U1 STM32F405RGT6, U2 SN65HVD230, U3 PowerIn, U4 LDL1117-3.3, U5 RFM95W-915S2, U6 Bosch BMP388, U7 LSM6DS3TR-C, U8 W25Q128JVP, U9 H3LIS331DL, Y1 8mhz

Commit message: added SD card middle ware from cubemx
Parts:
- moved R29 24.9 mm to (178.0, 98.0), turned to 90 degrees
- moved R28 1.06 mm to (178.5, 92.5), turned to 90 degrees
- moved TP5 0.70 mm to (128.5, 104.3)
- moved BZ1 0.60 mm to (180.5, 110.0)
- moved J7 0.10 mm to (179.5, 56.3)
Routing:
- net /MCU/D+: track 2.02 -> 11.4 mm
- net /usb_type_c/D-: track 3.08 -> 11.9 mm
- net /usb_type_c/D+: track 8.64 -> 14.7 mm
- net /MCU/SWCLK: track 69.4 -> 68.2 mm
- net /Aux/IgnitionPower: track 44.8 -> 43.6 mm
