File: Schematics/AuxPyro.kicad_sch (KiCad schematic)
At the start: 8 parts, among them J2 Pyro, Q1 IRLML2502TRPBF

Commit message: dfm sent for ordering
Other:
- moved on the sheet: R21
Changed lines of the file:
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@@
 	(wire
 		(pts
-			(xy 130.81 93.98) (xy 119.38 93.98)
+			(xy 127 93.98) (xy 119.38 93.98)
 		)
 		(stroke
@@
 	(wire
 		(pts
-			(xy 144.78 93.98) (xy 138.43 93.98)
+			(xy 135.89 93.98) (xy 134.62 93.98)
 		)
 		(stroke
@@
 	(hierarchical_label "AuxADC"
 		(shape input)
-		(at 144.78 93.98 0)
+		(at 135.89 93.98 0)
 		(effects
 			(font
@@
 	(symbol
 		(lib_id "Device:R")
-		(at 134.62 93.98 90)
+		(at 130.81 93.98 90)
 		(unit 1)
 		(exclude_from_sim no)
@@
 		(fields_autoplaced yes)
 		(property "Reference" "R21"
-			(at 134.62 87.63 90)
+			(at 130.81 87.63 90)
 			(effects
 				(font
@@
 		)
 		(property "Value" "1k"
-			(at 134.62 90.17 90)
+			(at 130.81 90.17 90)
 			(effects
 				(font
@@
 		)
 		(property "Footprint" "Resistor_SMD:R_0805_2012Metric_Pad1.20x1.40mm_HandSolder"
-			(at 134.62 95.758 90)
+			(at 130.81 95.758 90)
 			(effects
 				(font
@@
 		)
 		(property "Datasheet" "~"
-			(at 134.62 93.98 0)
+			(at 130.81 93.98 0)
 			(effects
 				(font
@@
 		)
 		(property "Description" "Resistor"
-			(at 134.62 93.98 0)
+			(at 130.81 93.98 0)
 			(effects
 				(font
@@
 		)
 		(property "LCSC" "C95781"
-			(at 134.62 93.98 90)
-			(effects
-				(font
+			(at 130.81 93.98 90)
+			(effects
+				(font
